Commit message: Add files via upload

File: RUKA1/urdf/RUKA1.urdf (robot description, URDF)
Before this commit: robot RUKA1, 6 links, 5 joints
Links:
- link link2_link: geometry collision cylinder length=4.80740 radius=0.73101; visual mesh filename=../meshes/stl/ruka.010.stl scale=1.00000 1.00000 1.00000
Joints:
- joint link1_link_joint: limit lower=-1.00000 upper=1.00000 effort=0.00000 velocity=0.00000 -> lower=-2.00000 upper=2.00000 effort=0.00000 velocity=0.00000
- joint link2_link_joint: limit lower=-1.00000 upper=1.00000 effort=0.00000 velocity=0.00000 -> lower=-2.00000 upper=2.00000 effort=0.00000 velocity=0.00000
- joint link3_link_joint: limit lower=-1.00000 upper=1.00000 effort=0.00000 velocity=0.00000 -> lower=-2.00000 upper=2.00000 effort=0.00000 velocity=0.00000
