Commit message: Add files via upload

File: bobotURDF/urdf/bobot.urdf (robot description, URDF)
Before this commit: robot bobot, 13 links, 12 joints
Links:
- link body0_plast_white_link: geometry collision box size=7.90146 11.50936 13.78356; visual mesh filename=../meshes/stl/body_black.stl scale=1.00000 1.00000 1.00000
- link head_steel_link: geometry collision box size=4.85000 7.60360 10.34980; visual mesh filename=../meshes/stl/head_black.stl scale=1.00000 1.00000 1.00000
- link leftArm5_plast_link: geometry collision box size=2.00002 1.00000 2.27000; visual mesh filename=../meshes/stl/LAP5.stl scale=1.00000 1.00000 1.00000
- link rightArm5_red_link: geometry collision box size=2.40701 1.08017 2.52897; visual mesh filename=../meshes/stl/RAP5.stl scale=1.00000 1.00000 1.00000

Commit message: Add files via upload

File: bobotURDF/urdf/bobot.urdf (robot description, URDF)
Before this commit: robot bobot, 13 links, 12 joints
Links:
- link body0_plast_white_link: geometry collision box size=7.90146 5.05599 13.78356; collision box size=7.90146 6.90555 11.75249

Commit message: Add files via upload

File: bobotURDF/urdf/bobot.urdf (robot description, URDF)
Before this commit: robot bobot, 13 links, 12 joints
Links:
- link body0_plast_white_link: geometry visual mesh filename=../meshes/stl/body_black.stl scale=1.00000 1.00000 1.00000; visual mesh filename=../meshes/stl/body_red.stl scale=1.00000 1.00000 1.00000
- link head_steel_link: geometry collision mesh filename=../meshes/stl/Cube.004.stl scale=0.77813 1.10000 1.56125; visual mesh filename=../meshes/stl/head_black.stl scale=1.00000 1.00000 1.00000

Commit message: Add files via upload

File: bobotURDF/urdf/bobot.urdf (robot description, URDF)
Before this commit: robot bobot, 13 links, 12 joints
Links:
- link head_steel_link: geometry collision box size=5.33500 8.36396 11.24074; visual mesh filename=../meshes/stl/head_black.stl scale=1.00000 1.00000 1.00000

Commit message: Add files via upload

File: bobotURDF/urdf/bobot.urdf (robot description, URDF)
Before this commit: robot bobot, 13 links, 12 joints
Links:
- link body0_plast_white_link: geometry collision mesh filename=../meshes/stl/body_white.stl scale=1.00000 1.00000 1.00000; visual mesh filename=../meshes/stl/body_black.stl scale=1.00000 1.00000 1.00000
- link head_steel_link: geometry collision mesh filename=../meshes/stl/Cube.004.stl scale=0.77813 1.10000 1.56125; visual mesh filename=../meshes/stl/head_black.stl scale=1.00000 1.00000 1.00000

Commit message: Add files via upload

File: bobotURDF/urdf/bobot.urdf (robot description, URDF)
Before this commit: robot bobot, 13 links, 12 joints
Links:
- link body0_plast_white_link: geometry visual mesh filename=../meshes/stl/body_black.stl scale=1.00000 1.00000 1.00000; visual mesh filename=../meshes/stl/body_red.stl scale=1.00000 1.00000 1.00000

Commit message: Add files via upload

File: bobotURDF/urdf/bobot.urdf (robot description, URDF)
Before this commit: robot bobot, 13 links, 12 joints
Links:
- link head_steel_link: geometry collision mesh filename=../meshes/stl/Cube.004.stl scale=1.00000 1.00000 1.00000; visual mesh filename=../meshes/stl/head_black.stl scale=1.00000 1.00000 1.00000

Commit message: Add files via upload

File: bobotURDF/urdf/bobot.urdf (robot description, URDF)
Before this commit: robot bobot, 13 links, 12 joints
Links:
- link body0_plast_white_link: geometry collision box size=10.21537 21.71539 13.19779; collision box size=11.09341 23.58187 14.33216
- link head_steel_link: geometry collision mesh filename=../meshes/stl/Cube.001.stl scale=1.00000 1.00000 1.00000; collision mesh filename=../meshes/stl/Cube.004.stl scale=1.00000 1.00000 1.00000
- link leftArm5_plast_link: geometry visual mesh filename=../meshes/stl/LAP5.stl scale=1.00000 1.00000 1.00000; visual mesh filename=../meshes/stl/LAR5.stl scale=1.00000 1.00000 1.00000
- link rightArm5_red_link: geometry visual mesh filename=../meshes/stl/RAP5.stl scale=1.00000 1.00000 1.00000; visual mesh filename=../meshes/stl/RAR5.stl scale=1.00000 1.00000 1.00000
Joints:
- joint leftArm2_plast_link_joint: limit lower=-2.00000 upper=2.00000 effort=0.00000 velocity=0.00000 -> lower=-1.57000 upper=1.57000 effort=0.00000 velocity=0.00000
- joint rightArm2_link_joint: limit lower=-2.00000 upper=2.00000 effort=0.00000 velocity=0.00000 -> lower=-1.57000 upper=1.57000 effort=0.00000 velocity=0.00000

Commit message: Add files via upload

File: bobotURDF/urdf/bobot.urdf (robot description, URDF)
Before this commit: robot bobot, 13 links, 12 joints
Links:
- link body0_plast_white_link: geometry collision mesh filename=../meshes/stl/Cube.006.stl scale=1.00000 1.00000 1.00000; collision mesh filename=../meshes/stl/Cube.stl scale=1.00000 1.00000 1.00000

Commit message: Add files via upload

File: bobotURDF/urdf/bobot.urdf (robot description, URDF)
Before this commit: robot bobot, 13 links, 12 joints
Joints:
- joint head_steel_link_joint: limit lower=-0.80000 upper=0.80000 effort=0.00000 velocity=0.00000 -> lower=0.00000 upper=4.71200 effort=0.00000 velocity=0.00000
- joint leftArm1_link_joint: limit lower=-3.14000 upper=3.14000 effort=0.00000 velocity=0.00000 -> lower=0.00000 upper=4.71200 effort=0.00000 velocity=0.00000
- joint leftArm1_plast_link_joint: origin xyz=-0.00000 17.49999 -6.17249 rpy=0.00000 0.00000 0.00000 -> xyz=-0.00000 17.49999 -6.17249 rpy=0.00000 0.00000 1.57080
- joint neck_plast_link_joint: limit lower=-1.00000 upper=1.00000 effort=0.00000 velocity=0.00000 -> lower=0.00000 upper=4.71200 effort=0.00000 velocity=0.00000
- joint rightArm2_link_joint: limit lower=-1.57000 upper=1.57000 effort=0.00000 velocity=0.00000 -> lower=0.00000 upper=4.71200 effort=0.00000 velocity=0.00000
- joint rightArm3_link_joint: limit lower=-2.00000 upper=2.00000 effort=0.00000 velocity=0.00000 -> lower=0.00000 upper=4.71200 effort=0.00000 velocity=0.00000
- joint rightArm4_link_joint: limit lower=-2.00000 upper=2.00000 effort=0.00000 velocity=0.00000 -> lower=0.00000 upper=4.71200 effort=0.00000 velocity=0.00000
- joint rightArm5_plast_link_joint: limit lower=-3.14000 upper=3.14000 effort=0.00000 velocity=0.00000 -> lower=0.00000 upper=4.71200 effort=0.00000 velocity=0.00000

Commit message: Add files via upload

File: bobotURDF/urdf/bobot.urdf (robot description, URDF)
Before this commit: robot bobot, 13 links, 12 joints
Joints:
- joint head_steel_link_joint: origin xyz=0.00000 1.90250 -0.00500 rpy=0.00000 0.00000 0.00000 -> xyz=0.00483 1.90250 0.00127 rpy=0.00000 0.00000 0.00000
- joint leftArm1_plast_link_joint: limit lower=-3.14000 upper=3.14000 effort=0.00000 velocity=0.00000 -> lower=0.00000 upper=4.71000 effort=0.00000 velocity=0.00000; origin xyz=-0.00000 17.49999 -6.17249 rpy=0.00000 0.00000 1.57080 -> xyz=-0.00000 17.49999 -6.17249 rpy=0.00000 0.00000 0.00000
- joint leftArm2_plast_link_joint: limit lower=-1.57000 upper=1.57000 effort=0.00000 velocity=0.00000 -> lower=0.00000 upper=4.71000 effort=0.00000 velocity=0.00000; origin xyz=-0.00500 -0.00000 -1.87501 rpy=0.00000 0.00000 0.00000 -> xyz=-0.00439 0.00239 -1.87501 rpy=0.00000 0.00000 0.00000
- joint leftArm3_plast_link_joint: limit lower=-2.00000 upper=2.00000 effort=0.00000 velocity=0.00000 -> lower=0.00000 upper=4.71000 effort=0.00000 velocity=0.00000; origin xyz=0.00000 0.00000 -3.20000 rpy=0.00000 0.00000 0.00000 -> xyz=-1.25957 -2.30830 1.82353 rpy=-0.00000 -0.00000 0.00000
- joint leftArm4_link_joint: limit lower=-2.00000 upper=2.00000 effort=0.00000 velocity=0.00000 -> lower=0.00000 upper=4.71000 effort=0.00000 velocity=0.00000; origin xyz=-0.00000 -0.00000 -3.20000 rpy=0.00000 0.00000 0.00000 -> xyz=1.44299 2.64443 1.07923 rpy=0.00000 -0.00000 0.00000
- joint leftArm5_plast_link_joint: limit lower=-3.14000 upper=3.14000 effort=0.00000 velocity=0.00000 -> lower=0.00000 upper=4.71000 effort=0.00000 velocity=0.00000; origin xyz=0.00500 -0.00000 -1.32502 rpy=0.00000 0.00000 0.00000 -> xyz=-0.48906 -0.90669 0.83332 rpy=0.00000 -0.00000 -0.00000
- joint rightArm2_link_joint: origin xyz=-0.00500 0.00000 1.87501 rpy=0.00000 0.00000 0.00000 -> xyz=0.00132 0.00482 1.87501 rpy=0.00000 0.00000 0.00000
- joint rightArm3_link_joint: origin xyz=-0.00000 0.00000 3.20000 rpy=0.00000 0.00000 0.00000 -> xyz=1.99369 -0.54466 2.44307 rpy=0.00000 0.00000 -0.00000
- joint rightArm4_link_joint: origin xyz=-0.00000 0.00000 3.19999 rpy=0.00000 0.00000 0.00000 -> xyz=-2.38327 0.65110 -2.03372 rpy=0.00000 0.00000 0.00000
- joint rightArm5_plast_link_joint: origin xyz=0.00500 0.00000 1.32502 rpy=0.00000 0.00000 0.00000 -> xyz=0.05600 -0.02048 1.32369 rpy=-0.00000 0.00000 -0.00000

Commit message: Add files via upload

File: bobotURDF/urdf/bobot.urdf (robot description, URDF)
Before this commit: robot bobot, 13 links, 12 joints
Joints:
- joint head_steel_link_joint: origin xyz=0.00483 1.90250 0.00127 rpy=0.00000 0.00000 0.00000 -> xyz=0.00000 1.90250 -0.00500 rpy=0.00000 0.00000 0.00000
- joint leftArm1_plast_link_joint: origin xyz=-0.00000 17.49999 -6.17249 rpy=0.00000 0.00000 0.00000 -> xyz=-0.00000 17.49999 -6.17249 rpy=0.00000 0.00000 0.49951
- joint leftArm2_plast_link_joint: origin xyz=-0.00439 0.00239 -1.87501 rpy=0.00000 0.00000 0.00000 -> xyz=-0.00500 -0.00000 -1.87501 rpy=2.17712 0.00000 -0.00000
- joint leftArm3_plast_link_joint: origin xyz=-1.25957 -2.30830 1.82353 rpy=-0.00000 -0.00000 0.00000 -> xyz=0.00000 0.00000 -3.20000 rpy=2.19126 -0.00000 -0.00000
- joint leftArm4_link_joint: origin xyz=1.44299 2.64443 1.07923 rpy=0.00000 -0.00000 0.00000 -> xyz=-0.00000 -0.00000 -3.20000 rpy=-2.11743 -0.00000 -0.00000
- joint leftArm5_plast_link_joint: origin xyz=-0.48906 -0.90669 0.83332 rpy=0.00000 -0.00000 -0.00000 -> xyz=0.00500 -0.00000 -1.32502 rpy=-0.00000 -0.00000 0.51365
- joint rightArm2_link_joint: origin xyz=0.00132 0.00482 1.87501 rpy=0.00000 0.00000 0.00000 -> xyz=-0.00500 0.00000 1.87501 rpy=0.00000 0.00000 0.00000
- joint rightArm3_link_joint: origin xyz=1.99369 -0.54466 2.44307 rpy=0.00000 0.00000 -0.00000 -> xyz=-0.00000 0.00000 3.20000 rpy=0.00000 0.00000 0.00000
- joint rightArm4_link_joint: origin xyz=-2.38327 0.65110 -2.03372 rpy=0.00000 0.00000 0.00000 -> xyz=-0.00000 0.00000 3.19999 rpy=0.00000 0.00000 0.00000
- joint rightArm5_plast_link_joint: origin xyz=0.05600 -0.02048 1.32369 rpy=-0.00000 0.00000 -0.00000 -> xyz=0.00500 0.00000 1.32502 rpy=0.00000 0.00000 0.00000

Commit message: Add files via upload

File: bobotURDF/urdf/bobot.urdf (robot description, URDF)
Before this commit: robot bobot, 13 links, 12 joints
Joints:
- joint leftArm1_plast_link_joint: origin xyz=-0.00000 17.49999 -6.17249 rpy=0.00000 0.00000 0.49951 -> xyz=-0.00000 17.49999 -6.17249 rpy=0.00000 0.00000 -0.49951
- joint leftArm2_plast_link_joint: origin xyz=-0.00500 -0.00000 -1.87501 rpy=2.17712 0.00000 -0.00000 -> xyz=-0.00500 -0.00000 -1.87501 rpy=-2.17712 0.00000 0.00000
- joint leftArm3_plast_link_joint: origin xyz=0.00000 0.00000 -3.20000 rpy=2.19126 -0.00000 -0.00000 -> xyz=0.00000 0.00000 -3.20000 rpy=-2.19126 -0.00000 0.00000
- joint leftArm4_link_joint: origin xyz=-0.00000 -0.00000 -3.20000 rpy=-2.11743 -0.00000 -0.00000 -> xyz=-0.00000 -0.00000 -3.20000 rpy=2.11743 -0.00000 0.00000
- joint leftArm5_plast_link_joint: origin xyz=0.00500 -0.00000 -1.32502 rpy=-0.00000 -0.00000 0.51365 -> xyz=0.00500 -0.00000 -1.32502 rpy=0.00000 0.00000 -0.51365

Commit message: Add files via upload

File: bobotURDF/urdf/bobot.urdf (robot description, URDF)
Before this commit: robot bobot, 13 links, 12 joints
Joints:
- joint leftArm1_plast_link_joint: origin xyz=-0.00000 17.49999 -6.17249 rpy=0.00000 0.00000 -0.49951 -> xyz=-0.00000 17.49999 -6.17249 rpy=0.00000 0.00000 0.00000
- joint leftArm2_plast_link_joint: origin xyz=-0.00500 -0.00000 -1.87501 rpy=-2.17712 0.00000 0.00000 -> xyz=-0.00500 -0.00000 -1.87501 rpy=0.00000 0.00000 0.00000
- joint leftArm3_plast_link_joint: origin xyz=0.00000 0.00000 -3.20000 rpy=-2.19126 -0.00000 0.00000 -> xyz=0.00000 0.00000 -3.20000 rpy=0.00000 0.00000 0.00000
- joint leftArm4_link_joint: origin xyz=-0.00000 -0.00000 -3.20000 rpy=2.11743 -0.00000 0.00000 -> xyz=-0.00000 -0.00000 -3.20000 rpy=0.00000 0.00000 0.00000
- joint leftArm5_plast_link_joint: origin xyz=0.00500 -0.00000 -1.32502 rpy=0.00000 0.00000 -0.51365 -> xyz=0.00500 -0.00000 -1.32502 rpy=0.00000 0.00000 0.00000

Commit message: Add files via upload

File: bobotURDF/urdf/bobot.urdf (robot description, URDF)
Before this commit: robot bobot, 13 links, 12 joints
Joints:
- removed joint leftArm1_link_joint
- added joint rightArm1_link_joint: type revolute, parent body0_plast_white_link, child rightArm1_steel_link, origin xyz=0.00000 17.49999 6.17249 rpy=0.00000 0.00000 0.00000, axis 0.00000 0.00000 1.00000, limit lower=-1.83400 upper=1.83400 effort=0.00000 velocity=0.00000
- joint head_steel_link_joint: limit lower=0.00000 upper=4.71200 effort=0.00000 velocity=0.00000 -> lower=-1.83400 upper=1.83400 effort=0.00000 velocity=0.00000
- joint leftArm1_plast_link_joint: limit lower=0.00000 upper=4.71000 effort=0.00000 velocity=0.00000 -> lower=-1.83400 upper=1.83400 effort=0.00000 velocity=0.00000
- joint leftArm2_plast_link_joint: limit lower=0.00000 upper=4.71000 effort=0.00000 velocity=0.00000 -> lower=-1.83400 upper=1.83400 effort=0.00000 velocity=0.00000
- joint leftArm3_plast_link_joint: limit lower=0.00000 upper=4.71000 effort=0.00000 velocity=0.00000 -> lower=-1.83400 upper=1.83400 effort=0.00000 velocity=0.00000
- joint leftArm4_link_joint: limit lower=0.00000 upper=4.71000 effort=0.00000 velocity=0.00000 -> lower=-1.83400 upper=1.83400 effort=0.00000 velocity=0.00000
- joint leftArm5_plast_link_joint: limit lower=0.00000 upper=4.71000 effort=0.00000 velocity=0.00000 -> lower=-1.83400 upper=1.83400 effort=0.00000 velocity=0.00000; origin xyz=0.00500 -0.00000 -1.32502 rpy=0.00000 0.00000 0.00000 -> xyz=0.00500 -0.00000 -1.32502 rpy=-0.00000 0.00000 0.00000
- joint neck_plast_link_joint: limit lower=0.00000 upper=4.71200 effort=0.00000 velocity=0.00000 -> lower=-1.83400 upper=1.83400 effort=0.00000 velocity=0.00000
- joint rightArm2_link_joint: limit lower=0.00000 upper=4.71200 effort=0.00000 velocity=0.00000 -> lower=-1.83400 upper=1.83400 effort=0.00000 velocity=0.00000
- joint rightArm3_link_joint: limit lower=0.00000 upper=4.71200 effort=0.00000 velocity=0.00000 -> lower=-1.83400 upper=1.83400 effort=0.00000 velocity=0.00000
- joint rightArm4_link_joint: limit lower=0.00000 upper=4.71200 effort=0.00000 velocity=0.00000 -> lower=-1.83400 upper=1.83400 effort=0.00000 velocity=0.00000
- joint rightArm5_plast_link_joint: limit lower=0.00000 upper=4.71200 effort=0.00000 velocity=0.00000 -> lower=-1.83400 upper=1.83400 effort=0.00000 velocity=0.00000

Commit message: Add files via upload

File: bobotURDF/urdf/bobot.urdf (robot description, URDF)
Before this commit: robot bobot, 13 links, 12 joints
Joints:
- joint head_steel_link_joint: limit lower=-1.83400 upper=1.83400 effort=0.00000 velocity=0.00000 -> lower=-0.70000 upper=0.70000 effort=0.00000 velocity=0.00000
- joint leftArm1_plast_link_joint: limit lower=-1.83400 upper=1.83400 effort=0.00000 velocity=0.00000 -> lower=-0.26000 upper=3.40000 effort=0.00000 velocity=0.00000
- joint leftArm2_plast_link_joint: origin xyz=-0.00500 -0.00000 -1.87501 rpy=0.00000 0.00000 0.00000 -> xyz=0.00000 -0.00500 -1.87501 rpy=0.00000 0.00000 0.00000
- joint leftArm5_plast_link_joint: origin xyz=0.00500 -0.00000 -1.32502 rpy=-0.00000 0.00000 0.00000 -> xyz=0.00500 -0.00000 -1.32502 rpy=0.00000 0.00000 0.00000
- joint rightArm1_link_joint: limit lower=-1.83400 upper=1.83400 effort=0.00000 velocity=0.00000 -> lower=-0.26000 upper=3.10000 effort=0.00000 velocity=0.00000

Commit message: Add files via upload

File: bobotURDF/urdf/bobot.urdf (robot description, URDF)
Before this commit: robot bobot, 13 links, 12 joints
Links:
- added link Armature; visual mesh filename=../meshes/stl/Cube.001.stl scale=1.00000 1.00000 1.00000
Joints:
- added joint rArmEff_Link: type revolute, parent rightArm5_red_link, child Armature, origin xyz=0.50000 0.00000 2.29749 rpy=0.00000 0.00000 0.00000, axis 0.00000 1.00000 0.00000, limit lower=-3.14000 upper=3.14000 effort=0.00000 velocity=0.00000

Commit message: Add files via upload

File: bobotURDF/urdf/bobot.urdf (robot description, URDF)
Before this commit: robot bobot, 14 links, 13 joints
Links:
- removed link Armature
- added link HeadEff_link; visual mesh filename=../meshes/stl/Cube.040.stl scale=1.00000 1.00000 1.00000
- added link lArmEff_link; visual mesh filename=../meshes/stl/LAP5.001.stl scale=1.00000 1.00000 1.00000
- added link rArmEff_link; visual mesh filename=../meshes/stl/Cube.001.stl scale=1.00000 1.00000 1.00000
Joints:
- removed joint head_steel_link_joint
- removed joint leftArm1_plast_link_joint
- removed joint leftArm4_link_joint
- added joint HeadEff_joint: type revolute, parent head_steel_link, child HeadEff_link, origin xyz=2.10444 3.65079 0.00500 rpy=0.00000 0.00000 0.00000, axis 0.00000 0.00000 1.00000, limit lower=-3.14000 upper=3.14000 effort=0.00000 velocity=0.00000
- added joint lArmEff_joint: type revolute, parent leftArm5_plast_link, child lArmEff_link, origin xyz=0.50000 0.00000 -2.89749 rpy=0.00000 0.00000 0.00000, axis 0.00000 1.00000 0.00000, limit lower=-3.14000 upper=3.14000 effort=0.00000 velocity=0.00000
- added joint leftArm1_plast_joint: type revolute, parent body0_plast_white_link, child leftArm1_plast_link, origin xyz=-0.00000 17.49999 -6.17249 rpy=0.00000 0.00000 0.00000, axis 0.00000 0.00000 1.00000, limit lower=-0.05480 upper=0.05480 effort=0.00000 velocity=0.00000
- added joint leftArm4_Joint: type revolute, parent leftArm3_plast_link, child leftArm4_link, origin xyz=-0.00000 -0.00000 -3.20000 rpy=0.00000 0.00000 0.00000, axis 1.00000 0.00000 0.00000, limit lower=-0.05480 upper=0.05480 effort=0.00000 velocity=0.00000
- added joint rArmEff_joint: type revolute, parent rightArm5_red_link, child rArmEff_link, origin xyz=0.50000 0.00000 2.89749 rpy=0.00000 0.00000 0.00000, axis 0.00000 1.00000 0.00000, limit lower=-3.14000 upper=3.14000 effort=0.00000 velocity=0.00000
- joint rArmEff_Link: axis 0.00000 1.00000 0.00000 -> 0.00000 0.00000 1.00000; child Armature -> head_steel_link; limit lower=-3.14000 upper=3.14000 effort=0.00000 velocity=0.00000 -> lower=-0.05480 upper=0.05480 effort=0.00000 velocity=0.00000; origin xyz=0.50000 0.00000 2.29749 rpy=0.00000 0.00000 0.00000 -> xyz=0.00000 1.90250 -0.00500 rpy=0.00000 0.00000 0.00000; parent rightArm5_red_link -> neck_plast_link

Commit message: Add files via upload

File: bobotURDF/urdf/bobot.urdf (robot description, URDF)
Before this commit: robot bobot, 16 links, 15 joints
Joints:
- removed joint rArmEff_Link
- added joint head_steel_Joint: type revolute, parent neck_plast_link, child head_steel_link, origin xyz=0.00000 1.90250 -0.00500 rpy=0.00000 0.00000 0.00000, axis 0.00000 0.00000 1.00000, limit lower=-0.05480 upper=0.05480 effort=0.00000 velocity=0.00000

Commit message: Add files via upload

File: bobotURDF/urdf/bobot.urdf (robot description, URDF)
Before this commit: robot bobot, 16 links, 15 joints
Joints:
- joint leftArm1_plast_joint: limit lower=-0.05480 upper=0.05480 effort=0.00000 velocity=0.00000 -> lower=-1.83000 upper=1.83000 effort=0.00000 velocity=0.00000

Commit message: Add files via upload

File: bobotURDF/urdf/bobot.urdf (robot description, URDF)
Before this commit: robot bobot, 16 links, 15 joints
Joints:
- joint head_steel_Joint: limit lower=-0.05480 upper=0.05480 effort=0.00000 velocity=0.00000 -> lower=-0.50000 upper=0.50000 effort=0.00000 velocity=0.00000
- joint lArmEff_joint: origin xyz=0.50000 0.00000 -2.89749 rpy=0.00000 0.00000 0.00000 -> xyz=0.00000 -0.50000 -2.89749 rpy=0.00000 0.00000 0.00000
- joint leftArm2_plast_link_joint: axis 1.00000 0.00000 0.00000 -> 0.00000 -1.00000 0.00000; origin xyz=0.00000 -0.00500 -1.87501 rpy=0.00000 0.00000 0.00000 -> xyz=-0.00500 -0.00000 -1.87501 rpy=0.00000 0.00000 0.00000
- joint leftArm3_plast_link_joint: axis 1.00000 0.00000 0.00000 -> 0.00000 -1.00000 0.00000
- joint leftArm4_Joint: axis 1.00000 0.00000 0.00000 -> 0.00000 -1.00000 0.00000; limit lower=-0.05480 upper=0.05480 effort=0.00000 velocity=0.00000 -> lower=-1.83000 upper=1.83000 effort=0.00000 velocity=0.00000; origin xyz=-0.00000 -0.00000 -3.20000 rpy=0.00000 0.00000 0.00000 -> xyz=-0.00000 0.00000 -3.20000 rpy=0.00000 0.00000 0.00000
- joint leftArm5_plast_link_joint: origin xyz=0.00500 -0.00000 -1.32502 rpy=0.00000 0.00000 0.00000 -> xyz=-0.00000 -0.00500 -1.32502 rpy=0.00000 0.00000 0.00000
- joint rArmEff_joint: origin xyz=0.50000 0.00000 2.89749 rpy=0.00000 0.00000 0.00000 -> xyz=0.00000 -0.50000 2.89749 rpy=0.00000 0.00000 0.00000
- joint rightArm1_link_joint: limit lower=-0.26000 upper=3.10000 effort=0.00000 velocity=0.00000 -> lower=-1.83000 upper=1.83000 effort=0.00000 velocity=0.00000
- joint rightArm2_link_joint: axis 1.00000 0.00000 0.00000 -> 0.00000 1.00000 0.00000; origin xyz=-0.00500 0.00000 1.87501 rpy=0.00000 0.00000 0.00000 -> xyz=-0.00000 0.00500 1.87501 rpy=0.00000 0.00000 0.00000
- joint rightArm3_link_joint: axis 1.00000 0.00000 0.00000 -> 0.00000 1.00000 0.00000; origin xyz=-0.00000 0.00000 3.20000 rpy=0.00000 0.00000 0.00000 -> xyz=0.00000 0.00000 3.20000 rpy=0.00000 0.00000 0.00000
- joint rightArm4_link_joint: axis 1.00000 0.00000 0.00000 -> 0.00000 1.00000 0.00000; origin xyz=-0.00000 0.00000 3.19999 rpy=0.00000 0.00000 0.00000 -> xyz=0.00000 0.00000 3.19999 rpy=0.00000 0.00000 0.00000
- joint rightArm5_plast_link_joint: origin xyz=0.00500 0.00000 1.32502 rpy=0.00000 0.00000 0.00000 -> xyz=0.00000 -0.00500 1.32502 rpy=0.00000 0.00000 0.00000

Commit message: Add files via upload

File: bobotURDF/urdf/bobot.urdf (robot description, URDF)
Before this commit: robot bobot, 16 links, 15 joints
Links:
- link rArmEff_link: geometry visual box size=1.00000 1.00000 1.00000
